Commit message: Complete CTC

File: src/universal_robot/ur_description/urdf/inc/ur_macro.xacro (robot description, xacro)
@@ -316,6 +316,4 @@
       <child link="${prefix}tool0"/>
     </joint>
-    <xacro:include filename="$(find robotiq_85_description)/urdf/robotiq_85_gripper.urdf.xacro" />
-    <xacro:robotiq_85_gripper gripper_prefix="" parent="${prefix}tool0"/>
   </xacro:macro>
 </robot>

File: src/universal_robot/ur_gazebo/urdf/ur.xacro (robot description, xacro)
@@ -65,5 +65,5 @@
     <parent link="world"/>
     <child link="base_link"/>
-    <origin xyz="0 0 1" rpy="0 0 0"/>
+    <origin xyz="0 0 0" rpy="0 0 0"/>
   </joint>
   <link name="tool0_controller"/>
